File: bbstack.sch (KiCad schematic (older format))
At the start: 4 parts, among them J1 CONN_01X17, J2 CONN_01X16, J3 CONN_01X17, J4 CONN_01X16

Commit message: Update to rev1.1
Parts:
- added J10, J11, J12, J13, J14, J15, J16, J17, J18, J19, J20, J5, J6, J7, J8, J9: CONN_01X14, common:Pin_Header_Straight_1x14_Pitch2.54mm, symbol CONN_01X14
- added J21: CONN_01X03, common:Pin_Header_Straight_1x03_Pitch2.54mm, symbol CONN_01X03
- added J22: grove_01X04, Connectors:Grove_1x04, symbol CONN_01X04
Connections:
- new net: J22.1 (P1), J8.2 (P2)
- new net: J22.2 (P2), J8.3 (P3)
- new net: J22.3 (P3), J8.4 (P4)
- new net: J22.4 (P4), J8.5 (P5)
- new net: J21.3 (P3), J8.7 (P7)
- new net: J21.2 (P2), J8.8 (P8)
- new net: J21.1 (P1), J8.9 (P9)
- no-connect marks 1 -> 218
