File: emptystack.sch (KiCad schematic (older format))
At the start: 22 parts, among them J1 CONN_01X17, J10 CONN_01X14, J11 CONN_01X14, J12 CONN_01X14, J13 CONN_01X14, J14 CONN_01X14, J15 CONN_01X14, J16 CONN_01X14, J17 CONN_01X14, J18 CONN_01X14, J19 CONN_01X14, J2 CONN_01X16, J20 CONN_01X14, J21 CONN_01X03, J22 grove_01X04, J3 CONN_01X17, J4 CONN_01X16, J5 CONN_01X14, J6 CONN_01X14, J7 CONN_01X14, J8 CONN_01X14, J9 CONN_01X14

Commit message: Change file names to emptystack
Parts:
- J21: footprint Pin_Headers:Pin_Header_Straight_1x03_Pitch2.54mm -> common:Pin_Header_Straight_1x03_Pitch2.54mm
Connections:
- net at J8.10 (P10): no longer J21.1 (P1)
- net at J8.7 (P7): now also J21.3 (P3)
- net at J8.8 (P8): now also J21.2 (P2); no longer J21.3 (P3)
- net at J8.9 (P9): now also J21.1 (P1); no longer J21.2 (P2)
Other:
- moved on the sheet: J21
Changed lines of the file:
@@
 EESchema Schematic File Version 2
-LIBS:bbstack-rescue
+LIBS:emptystack-rescue
 LIBS:power
 LIBS:device
@@
 LIBS:MiscellaneousDevices
 LIBS:CP2102
-LIBS:bbstack-cache
+LIBS:emptystack-cache
 EELAYER 25 0
 EELAYER END
@@
 encoding utf-8
 Sheet 1 1
-Title "Bbstack"
+Title "EmptyStack"
 Date "2017-04-28"
 Rev "1.1"
 Comp ""
 Comment1 "by asukiaaa"
-Comment2 "github.com/asukiaaa/bbstack"
+Comment2 "github.com/asukiaaa/emptystack"
 Comment3 ""
 Comment4 ""
@@
 IO15
 $Comp
-L +3.3V #PWR1
+L +3.3V #PWR01
 U 1 1 58948A12
 P 1200 3050
-F 0 "#PWR1" H 1200 2900 50  0001 C CNN
+F 0 "#PWR01" H 1200 2900 50  0001 C CNN
 F 1 "+3.3V" H 1200 3190 50  0000 C CNN
 F 2 "" H 1200 3050 50  0000 C CNN
@@
 $EndComp
 $Comp
-L GND #PWR2
+L GND #PWR02
 U 1 1 58948B03
 P 1350 2600
-F 0 "#PWR2" H 1350 2350 50  0001 C CNN
+F 0 "#PWR02" H 1350 2350 50  0001 C CNN
 F 1 "GND" H 1350 2450 50  0000 C CNN
 F 2 "" H 1350 2600 50  0000 C CNN
@@
 $EndComp
 $Comp
-L GND #PWR6
+L GND #PWR03
 U 1 1 58948C68
 P 2750 4550
-F 0 "#PWR6" H 2750 4300 50  0001 C CNN
+F 0 "#PWR03" H 2750 4300 50  0001 C CNN
 F 1 "GND" H 2750 4400 50  0000 C CNN
 F 2 "" H 2750 4550 50  0000 C CNN
@@
 $EndComp
 $Comp
-L VCC #PWR4
+L VCC #PWR04
 U 1 1 58948CFD
 P 1350 4900
-F 0 "#PWR4" H 1350 4750 50  0001 C CNN
+F 0 "#PWR04" H 1350 4750 50  0001 C CNN
 F 1 "VCC" H 1350 5050 50  0000 C CNN
 F 2 "" H 1350 4900 50  0000 C CNN
@@
 $EndComp
 $Comp
-L +3.3V #PWR5
+L +3.3V #PWR05
 U 1 1 58948E57
 P 2750 4450
-F 0 "#PWR5" H 2750 4300 50  0001 C CNN
+F 0 "#PWR05" H 2750 4300 50  0001 C CNN
 F 1 "+3.3V" H 2750 4590 50  0000 C CNN
 F 2 "" H 2750 4450 50  0000 C CNN
@@
 $EndComp
 $Comp
-L GND #PWR3
+L GND #PWR06
 U 1 1 58948EC3
 P 1350 4450
-F 0 "#PWR3" H 1350 4200 50  0001 C CNN
+F 0 "#PWR06" H 1350 4200 50  0001 C CNN
 F 1 "GND" H 1350 4300 50  0000 C CNN
 F 2 "" H 1350 4450 50  0000 C CNN
@@
 NoConn ~ 6700 5650
 NoConn ~ 6700 5750
-$Comp
-L CONN_01X14 J8
-U 1 1 58F9E554
-P 5300 6650
-F 0 "J8" H 5300 7400 50  0000 C CNN
-F 1 "CONN_01X14" V 5400 6650 50  0000 C CNN
-F 2 "common:Pin_Header_Straight_1x14_Pitch2.54mm" H 5300 6650 50  0001 C CNN
-F 3 "" H 5300 6650 50  0001 C CNN
-	1    5300 6650
-	1    0    0    -1
-$EndComp
 NoConn ~ 5100 6000
 NoConn ~ 5100 6500
-NoConn ~ 5100 6600
+NoConn ~ 5100 6900
 NoConn ~ 5100 7000
 NoConn ~ 5100 7100
@@
 L CONN_01X03 J21
 U 1 1 59034F24
-P 4800 6800
-F 0 "J21" H 4800 7000 50  0000 C CNN
-F 1 "CONN_01X03" V 4900 6800 50  0000 C CNN
-F 2 "Pin_Headers:Pin_Header_Straight_1x03_Pitch2.54mm" H 4800 6800 50  0001 C CNN
-F 3 "" H 4800 6800 50  0001 C CNN
-	1    4800 6800
+P 4800 6700
+F 0 "J21" H 4800 6900 50  0000 C CNN
+F 1 "CONN_01X03" V 4900 6700 50  0000 C CNN
+F 2 "common:Pin_Header_Straight_1x03_Pitch2.54mm" H 4800 6700 50  0001 C CNN
+F 3 "" H 4800 6700 50  0001 C CNN
+	1    4800 6700
 	-1   0    0    1
 $EndComp
 Wire Wire Line
+	5000 6600 5100 6600
+Wire Wire Line
 	5000 6700 5100 6700
 Wire Wire Line
 	5000 6800 5100 6800
-Wire Wire Line
-	5000 6900 5100 6900
+$Comp
+L CONN_01X14 J8
+U 1 1 58F9E554
+P 5300 6650
+F 0 "J8" H 5300 7400 50  0000 C CNN
+F 1 "CONN_01X14" V 5400 6650 50  0000 C CNN
+F 2 "common:Pin_Header_Straight_1x14_Pitch2.54mm" H 5300 6650 50  0001 C CNN
+F 3 "" H 5300 6650 50  0001 C CNN
+	1    5300 6650
+	1    0    0    -1
+$EndComp
 $EndSCHEMATC
